File: Esquematic_Maleter.kicad_sch (KiCad schematic)
At the start: 52 parts, among them J1 Conn_01x02, J3 Conn_01x02, J4 Conn_01x02, J5 Conn_01x06_Fem, K1 ADW11, Q1 BC817, U1 MCP2551-I-P, U2 LM1117-5.0, U3 LM1117-3.3, U4 FDC2212QDNTTQ1, U5 PIC18F258-I/SP, U6 AD8616ARZ, Y1 Crystal

Commit message: Add files via upload
Parts:
- removed J?: Conn_01x03_Male, symbol Connector:Conn_01x03_Male
- removed S? (x2): 2-1437565-7, Llibreria_Prac3:SW_2-1437565-7, symbol Llibreria_Prac3:2-1437565-7
- removed U3: LM1117-3.3, BQ_Library:TO254P1054X470X1955-3, symbol Regulator_Linear:LM1117-3.3
- added D3, D4, D5: LED, symbol Device:LED
- added J6: conn, symbol Connector:Conn_01x04_Male
- added Q2, Q3: BC817, Package_TO_SOT_SMD:SOT-23, symbol Transistor_BJT:BC817
- added R12, R13: R, Resistor_SMD:R_1206_3216Metric, symbol Device:R_US
- added R15: R, symbol Device:R_Small_US
- added U2: LM1117-3.3, BQ_Library:TO254P1054X470X1955-3, symbol Regulator_Linear:LM1117-3.3
- C2: value c -> 33pF
- C3: value c1 -> 33pF
- L1, L2: value L -> 18uH
- gave numbers to parts that had none: 10
- renumbered U2 to U1, U1 to U3
Connections:
- net +VCC1: now also R12.1
- net +VCC2: now also R13.1, U2.2 (VO)
- net GND: now also D3.1 (K), D4.1 (K), D5.1 (K), J6.2 (Pin_2), Q2.2 (E), Q3.2 (E), U2.1 (GND)
- net Heater: now also U5.25 (RB4); no longer U5.21 (RB0/INT0)
- net M1: now also J6.4 (Pin_4)
- net M2: now also J6.3 (Pin_3)
- net Vref: now reaches U6.6 (-INB)
- net Vref: now also J6.1 (Pin_1)
- net at C4.1, D2.1 (K): now also U2.3 (VI)
- net at D6.2 (A), K2.1: now also Q2.3 (C)
- net at D7.2 (A), K3.1: now also Q3.3 (C)
- net Relé1: now reaches U5.11 (RC0/T1OSO/T1CK1)
- net Relé1: now also Q2.1 (B)
- net Relé2: now reaches U5.12 (RC1/T1OSI)
- net Relé2: now also Q3.1 (B)
- net INTB: now reaches U5.22 (RB1/INT1)
- net INTB: now also U4.5 (INTB)
- net at U5.6 (RA4/T0CKI): now also R15.1
- net SD: now reaches U4.6 (SD)
- net SD: now also U5.21 (RB0/INT0)
- new net: D4.2 (A), R13.2
- new net: D5.2 (A), R15.2
- new net: D3.2 (A), R12.2
- no-connect marks 20 -> 16
Other:
- moved on the sheet: C1, C7, D1, R11, R9, U1

Commit message: Add files via upload
Parts:
- removed J6: conn, symbol Connector:Conn_01x04_Male
- added 1: TCA39306DTMR, symbol BQ_library:TCA39306DTMR
- added J6: Conn_Male, symbol Connector:Conn_01x03_Male
- added R16, R17, R21: 10k, symbol Device:R_Small_US
- added R18: 200k, symbol Device:R_Small_US
- added R19, R20: 22k, symbol Device:R_Small_US
- added R22: 80k, symbol Device:R_Small_US
Connections:
- net +VCC1: now also R16.2, R18.1, R19.1, R20.1
- net +VCC2: now also C8.1, R1.1, R2.1, U4.7 (VDD), 1.2 (VREF1), R21.1; no longer R1.2, R2.2
- net GND: now also J2.4, R7.1, 1.1 (GND), J6.1 (Pin_1), R17.1, R22.1; no longer U4.3 (CLKIN)
- net M1: now also J6.3 (Pin_3)
- net M2: now also J6.2 (Pin_2)
- net RX_CAN: no longer J2.7
- net TX_CAN: no longer J2.2
- net CANL: now reaches C9.2, R14.1, U3.6 (CANL)
- net CANL: now also J2.7
- net CANH: now reaches C9.1, R14.2, U3.7 (CANH)
- net CANH: now also J2.2
- net at U3.5 (Vref): now also R16.1, R17.2
- net Relé_Out: no longer names the net of K1.3, R6.1
- net Relé_Out: no longer R7.1
- removed net SCL: R1.1, U4.1 (SCL), U5.14 (RC3/SCK/SCL)
- removed net SDA: R2.1, U4.2 (SDA), U5.15 (RC4/SDI/SDA)
- net Vref: no longer names the net of U6.6 (-INB)
- net Vref: now also R21.2, R22.2
- new net: 1.7 (VREF2), 1.8 (EN), R18.2
- new net SCL1: 1.3 (SCL1), R1.2, U4.1 (SCL)
- new net SCL2: 1.6 (SCL2), R20.2, U5.14 (RC3/SCK/SCL)
- new net SDA1: 1.4 (SDA1), R2.2, U4.2 (SDA)
- new net SDA2: 1.5 (SDA2), R19.2, U5.15 (RC4/SDI/SDA)
- no-connect marks 16 -> 14
Other:
- note added: "Battery"
- note added: "Button for the heater"
- note added: "Level Shifter"
- note added: "Manual reset"
- note added: "Microcontroller"
- note added: "Oscillator"
- note added: "Programming connectors"
- note added: "Proximity sensor"
- note added: "Relays + BJT"
- note added: "Relays micro K"
- note added: "Resistant heater"
- note added: "Shunt and OpAmp"
- note added: "Tension regulators"
- note removed: "BATERIA"
- note removed: "Botonera per a la calefació"
- note removed: "Connectors de programació"
- note removed: "Driver"
- note removed: "Microcontrolador"
- note removed: "Oscil·lador"
- note removed: "Reguladors de tensió"
- note removed: "Relé + BJT"
- note removed: "Reset manual"
- note removed: "Resistència calefactora"
- note removed: "Sensor de proximitat"
- note removed: "Shunt & OpAmp"
- moved on the sheet: C11, C12, C13, C2, C3, C5, C8, C9, J2, J3, J4, L2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

Commit message: Add files via upload
Parts:
- removed 1: TCA39306DTMR, symbol BQ_library:TCA39306DTMR
- removed C11: 0.1uF, symbol Device:C_Small
- removed C13: 15 pF, Capacitor_SMD:C_0805_2012Metric, symbol Device:C
- removed C14: 100nF, Capacitor_THT:C_Radial_D4.0mm_H5.0mm_P1.50mm, symbol Device:C_Small
- removed R10, R11: 100k, symbol Device:R_Small_US
- removed R12: R, Resistor_SMD:R_1206_3216Metric, symbol Device:R_US
- removed R14: 60, symbol Device:R_Small_US
- removed R16: 10k, symbol Device:R_Small_US
- removed R2: 22k, symbol Device:R_Small_US
- removed R3, R5: 10K, Resistor_SMD:R_1206_3216Metric, symbol Device:R_US
- removed R6: Heater, symbol Device:Heater
- removed R7: R_Shunt, symbol Device:R_Shunt
- removed U1: LM1117-5.0, BQ_Library:TO254P1054X470X1955-3, symbol Regulator_Linear:LM1117-5.0
- removed U2: LM1117-3.3, BQ_Library:TO254P1054X470X1955-3, symbol Regulator_Linear:LM1117-3.3
- removed U3: MCP2551-I-P, Package_DIP:DIP-8_W7.62mm, symbol Interface_CAN_LIN:MCP2551-I-P
- removed U4: FDC2212QDNTTQ1, SON50P400X400X100-13N, symbol BQ_library:FDC2212QDNTTQ1
- removed U5: PIC18F258-I/SP, DIP787W45P254L3556H508Q28, symbol BQ_library:PIC18F258-I{brace}slash}SP
- removed U6: AD8616ARZ, SOIC127P600X175-8N, symbol BQ_library:AD8616ARZ
- added C10: 0.1uF, Capacitor_SMD:C_0805_2012Metric_Pad1.18x1.45mm_HandSolder, symbol Device:C_Small
- added C11: 15 pF, Capacitor_SMD:C_0805_2012Metric, symbol Device:C
- added C13: 100nF, Capacitor_THT:C_Radial_D4.0mm_H5.0mm_P1.50mm, symbol Device:C_Small
- added J7: Conn_01x02, Connector_PinHeader_2.54mm:PinHeader_1x02_P2.54mm_Vertical, symbol Connector_Generic:Conn_01x02
- added R10, R11: 1k, Resistor_SMD:R_1206_3216Metric, symbol Device:R_US
- added R12: 60, Resistor_SMD:R_1206_3216Metric, symbol Device:R_Small_US
- added R2: 10K, Resistor_SMD:R_1206_3216Metric, symbol Device:R_US
- added R3: 22k, Resistor_SMD:R_1206_3216Metric, symbol Device:R_Small_US
- added R5: 10k, Resistor_SMD:R_1206_3216Metric, symbol Device:R_Small_US
- added R6: 200k, Resistor_SMD:R_1206_3216Metric, symbol Device:R_Small_US
- added R7: 20k, Resistor_SMD:R_1206_3216Metric, symbol Device:R_Small_US
- added Rshunt1: 2m, Llibreria_Projecte_Maleter:ShuntRes, symbol Device:R
- added U1: TCA39306DTMR, Llibreria_Projecte_Maleter:TCA39306DTMR, symbol BQ_library:TCA39306DTMR
- added U2: MCP2551-I-P, Package_DIP:DIP-8_W7.62mm, symbol Interface_CAN_LIN:MCP2551-I-P
- added U3: LM1117-5.0, BQ_Library:TO254P1054X470X1955-3, symbol Regulator_Linear:LM1117-5.0
- added U4: LM1117-3.3, BQ_Library:TO254P1054X470X1955-3, symbol Regulator_Linear:LM1117-3.3
- added U5: FDC2212QDNTTQ1, Llibreria_Projecte_Maleter:SON50P400X400X100-13N, symbol BQ_library:FDC2212QDNTTQ1
- added U6: PIC18F258-I/SP, Llibreria_Projecte_Maleter:DIP787W45P254L3556H508Q28, symbol BQ_library:PIC18F258-I{brace}slash}SP
- added U7: AD8616ARZ, Llibreria_Projecte_Maleter:SOIC127P600X175-8N, symbol BQ_library:AD8616ARZ
- C1: value 10uF -> 33pF
- C2: footprint (none) -> Capacitor_SMD:C_0805_2012Metric_Pad1.18x1.45mm_HandSolder
- C3: value 33pF -> 100nF; footprint (none) -> Capacitor_THT:C_Radial_D4.0mm_H5.0mm_P1.50mm
- C5: value 100nF -> 10uF; footprint Capacitor_THT:C_Radial_D4.0mm_H5.0mm_P1.50mm -> Capacitor_SMD:C_0805_2012Metric_Pad1.18x1.45mm_HandSolder
- C8: value 0.1 uF -> 100pF; footprint (none) -> Capacitor_THT:C_Radial_D4.0mm_H5.0mm_P1.50mm
- C9: value 100pF -> 0.1 uF; footprint Capacitor_THT:C_Radial_D4.0mm_H5.0mm_P1.50mm -> Capacitor_SMD:C_0805_2012Metric_Pad1.18x1.45mm_HandSolder
- D3, D4, D5: footprint (none) -> LED_THT:LED_D5.0mm
- J2: footprint (none) -> Connector_Dsub:DSUB-9_Male_Vertical_P2.77x2.84mm
- J3, J4: footprint (none) -> Connector_PinHeader_2.54mm:PinHeader_1x02_P2.54mm_Vertical
- J5: footprint (none) -> Connector_PinHeader_2.54mm:PinHeader_1x06_P2.54mm_Vertical
- J6: footprint (none) -> Connector_PinHeader_2.54mm:PinHeader_1x03_P2.54mm_Vertical
- K2, K3: footprint RELAY_1393280-5 -> Llibreria_Projecte_Maleter:RELAY_1393280-5
- L1, L2: footprint (none) -> Inductor_THT:L_Axial_L5.3mm_D2.2mm_P7.62mm_Horizontal_Vishay_IM-1
- R1: footprint (none) -> Resistor_SMD:R_1206_3216Metric
- R13: value R -> 10K
- R15: value R -> 1k; footprint (none) -> Resistor_SMD:R_1206_3216Metric
- R17: value 10k -> 1k; footprint (none) -> Resistor_SMD:R_1206_3216Metric
- R18: value 200k -> 1k; footprint (none) -> Resistor_SMD:R_1206_3216Metric
- R19: value 22k -> 100k; footprint (none) -> Resistor_SMD:R_1206_3216Metric
- R20: value 22k -> 10k; footprint (none) -> Resistor_SMD:R_1206_3216Metric
- R21: value 10k -> 100k; footprint (none) -> Resistor_SMD:R_1206_3216Metric
- R22: footprint (none) -> Resistor_SMD:R_1210_3225Metric
- R4: value Rext -> 10k; footprint (none) -> Resistor_SMD:R_1206_3216Metric
- R8, R9: value 1k -> 22k; footprint (none) -> Resistor_SMD:R_1206_3216Metric
- S1, S2: footprint Llibreria_Prac3:SW_2-1437565-7 -> Llibreria_Projecte_Maleter:SW_2-1437565-7
Connections:
- net SCL1 is gone; now on net GND: R1.2
- net SDA2 is gone; now on net IN_B: R19.2
- net +VCC1: now also C3.1, C6.1, R13.1, R4.2, R8.1, R9.1, C13.1, R10.1, R2.1, R6.1, U2.3 (VDD), U3.2 (VO), U6.20 (VDD), U7.8 (V+); no longer C5.1, C7.1, R18.1, R19.1, R20.1
- net CANH: now also C8.1, R12.2, U2.7 (CANH); no longer C9.1
- net CANL: now also C8.2, R12.1, U2.6 (CANL); no longer C9.2
- net GND: now also C7.1, C9.1, C9.2, R1.1, R17.2, R20.1, R21.1, C10.1, C10.2, C11.2, C13.2, J7.2 (Pin_2), R11.1, R3.1, R3.2, R5.1, R7.1, Rshunt1.2, U1.1 (GND), U1.2 (VREF1), U1.3 (SCL1), U1.4 (SDA1), U2.2 (VSS), U3.1 (GND), U4.1 (GND), U4.2 (VO), U5.1 (SCL), U5.10 (IN0B), U5.12 (IN1B), U5.2 (SDA), U5.4 (ADDR), U5.7 (VDD), U5.8 (GND), U6.19 (VSS), U6.8 (VSS), U7.4 (V-); no longer C8.2, Q2.2 (E), R17.1, R4.1
- net Heater: now also S1.1, S1.2, R2.2, U6.25 (RB4); no longer S2.1, S2.2
- net INTB: now also U5.5 (INTB), U6.22 (RB1/INT1)
- net IN_B: now also U7.1 (OUT_A), U7.5 (+INB)
- net M1: now also J6.2 (Pin_2); no longer J6.3 (Pin_3)
- net M2: now also J6.3 (Pin_3); no longer J6.2 (Pin_2)
- net OSC1: now also C11.1, U6.9 (OSC1/CLKI); no longer C12.1
- net OSC2 : now also C12.1, U6.10 (OSC2/CLKO/RA6)
- net PGC: now also U6.27 (RB6/PGC)
- net PGD: now also U6.28 (RB7/PGD)
- net PMW_5V: now also U6.13 (RC2/CCP1)
- net RESET: now also R13.2, S2.1, S2.2; no longer S1.1, S1.2
- net RX_CAN: now also U2.4 (RXD), U6.18 (RC7/RX/DT)
- net Relé1: now also U6.11 (RC0/T1OSO/T1CK1)
- net Relé2: now also U6.12 (RC1/T1OSI)
- net SCL2: now also R8.2, R9.2, R6.2, U1.5 (SDA2), U1.6 (SCL2), U1.7 (VREF2), U1.8 (EN), U6.14 (RC3/SCK/SCL), U6.15 (RC4/SDI/SDA); no longer R20.2
- net SD: now also U5.6 (SD), U6.21 (RB0/INT0)
- net TX_CAN: now also U2.1 (TXD), U6.17 (RC6/TX/CK)
- net VOUT: now also U6.2 (RA0/AN0/CVREF), U7.7 (OUT_B)
- net /MCLR: now also U6.1 (~{MCLR/VPP})
- net at R22.2: now also R20.2, U7.6 (-INB); no longer R21.2
- net at K1.3: now also J7.1 (Pin_1)
- net Relé_Out: now reaches R18.2
- net Relé_Out: now also Q2.2 (E), Rshunt1.1
- net at J3.2 (Pin_2), L1.1: now also C1.1, U5.9 (IN0A); no longer C2.1
- net at D4.2 (A): now also R11.2; no longer R13.2
- net at C4.1: now also D1.1 (K), U3.3 (VI); no longer D2.1 (K)
- net at D3.2 (A): now also R10.2
- net at J4.2 (Pin_2), L2.1: now also C2.1, U5.11 (IN1A); no longer C3.1
- net at R15.1: now also U6.6 (RA4/T0CKI)
- removed net +VCC2: C6.1, C8.1, R1.1, R13.1, R21.1
- new net: R4.1, R5.2, U2.5 (Vref)
- new net: C5.1, D2.1 (K), U4.3 (VI)
- new net: R17.1, R19.1, U7.2 (-INA)
- new net: R18.1, R21.2, U7.3 (+INA)
- new net: R7.2, U2.8 (Rs)
Other:
- title: PROJECTE EDD: Maleter -> Projecte EDD: Maleter

Commit message: Add files via upload
Parts:
- removed R4, R5: 10k, Resistor_SMD:R_1206_3216Metric, symbol Device:R_Small_US
- added C14: 100 nF, Capacitor_SMD:C_0805_2012Metric, symbol Device:C
- added D8: 1N4002, Diode_THT:D_5W_P10.16mm_Horizontal, symbol Diode:1N4002
- added R14, R23, R4: 60k, Resistor_SMD:R_1206_3216Metric, symbol Device:R_US
- added R16, R24, R5: 10k, Resistor_SMD:R_1206_3216Metric, symbol Device:R_US
Connections:
- net /MCLR is gone; now on net RESET: J5.1 (Pin_1), U6.1 (~{MCLR/VPP})
- net +VCC1: now also C14.1; no longer U7.8 (V+)
- net GND: now also U5.3 (CLKIN), R16.2, R24.1, R5.2; no longer C1.2, C10.1, C2.2, C7.1, C9.1, L1.2, L2.2, R1.1, R1.2, R11.1, R20.1, R3.1, R3.2, U1.2 (VREF1), U1.3 (SCL1), U1.4 (SDA1), U4.2 (VO), U5.1 (SCL), U5.10 (IN0B), U5.12 (IN1B), U5.2 (SDA), U5.4 (ADDR), U5.7 (VDD)
- net M1: now also K2.4; no longer K2.3
- net M2: now also K3.4; no longer K3.3
- net PMW_5V: now also R4.2; no longer Q1.1 (B)
- net Relé1: now also R14.2; no longer Q2.1 (B)
- net Relé2: now also R23.2; no longer Q3.1 (B)
- net SCL2: no longer R6.2, R8.2, U1.5 (SDA2), U1.7 (VREF2), U1.8 (EN), U6.15 (RC4/SDI/SDA)
- net VBAT: now also K2.3, K3.3, D8.1 (K); no longer D6.1 (K), D7.1 (K), K2.2, K2.4, K3.2, K3.4
- net at K1.1, Q1.3 (C): now also D8.2 (A)
- net VOUT renamed INTERRP
- new net: D6.1 (K), K2.2
- new net: Q3.1 (B), R23.1, R24.2
- new net: D7.1 (K), K3.2
- new net: C1.2, L1.2, U5.10 (IN0B)
- new net: C2.2, L2.2, U5.12 (IN1B)
- new net: Q2.1 (B), R14.1, R16.1
- new net: Q1.1 (B), R4.1, R5.1
- new net: C14.2, U7.8 (V+)
- new net: R6.2, U1.7 (VREF2), U1.8 (EN)
- new net +VCC2: C10.1, C7.1, C9.1, R1.1, R11.1, R20.1, R3.1, U1.2 (VREF1), U4.2 (VO), U5.4 (ADDR), U5.7 (VDD)
- new net SCL1: R1.2, U1.3 (SCL1), U5.1 (SCL)
- new net SDA1: R3.2, U1.4 (SDA1), U5.2 (SDA)
- new net SDA2: R8.2, U1.5 (SDA2), U6.15 (RC4/SDI/SDA)
- no-connect marks 14 -> 15
Other:
- moved on the sheet: D7, Q1
