File: Esquematic_Maleter.kicad_sch (KiCad schematic)
At the start: 72 parts, among them J1 Conn_01x02, J2 DB9_Male, J3 Conn_01x02, J4 Conn_01x02, J5 Conn_01x06_Fem, J6 Conn_Male, J7 Conn_01x02, K1 ADW11, K2 1393280-5, K3 1393280-5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

Commit message: Add files via upload
Parts:
- U1: footprint Llibreria_Projecte_Maleter:TCA39306DTMR -> Llibreria_Projecte_Maleter:SOP50P310X90-8N
Changed lines of the file:
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@@
     (effects (font (size 2 2) (thickness 0.4) bold) (justify left bottom))
   )
-  (text "Relays + BJT\n" (at 180.34 121.92 0)
+  (text "Relays + BJT\n" (at 166.7764 116.6622 0)
     (effects (font (size 2 2) (thickness 0.4) bold) (justify left bottom))
   )
-  (text "Shunt and OpAmp\n" (at 241.3 165.1 0)
+  (text "Shunt and OpAmp\n" (at 240.8682 162.6108 0)
     (effects (font (size 2 2) (thickness 0.4) bold) (justify left bottom))
   )
@@
     (effects (font (size 2 2) (thickness 0.4) bold) (justify left bottom))
   )
-  (text "Proximity sensor\n" (at 63.5 134.62 0)
+  (text "Proximity sensor\n" (at 63.0682 132.1308 0)
     (effects (font (size 2 2) (thickness 0.4) bold) (justify left bottom))
   )
-  (text "Resistant heater" (at 154.94 157.48 0)
+  (text "Resistant heater" (at 153.2382 156.2608 0)
     (effects (font (size 1.5 1.5) (thickness 0.3) bold) (justify left bottom))
   )
@@
     (property "Reference" "U1" (id 0) (at 45.72 173.99 0))
     (property "Value" "TCA39306DTMR" (id 1) (at 45.72 176.53 0))
-    (property "Footprint" "Llibreria_Projecte_Maleter:TCA39306DTMR" (id 2) (at 30.48 185.42 0)
+    (property "Footprint" "Llibreria_Projecte_Maleter:SOP50P310X90-8N" (id 2) (at 30.48 185.42 0)
       (effects (font (size 1.27 1.27)) hide)
     )
@@
     )
     (path "/a1c125c8-44d7-4112-b6e9-722d8701036e"
-      (reference "U1") (unit 1) (value "TCA39306DTMR") (footprint "Llibreria_Projecte_Maleter:TCA39306DTMR")
+      (reference "U1") (unit 1) (value "TCA39306DTMR") (footprint "Llibreria_Projecte_Maleter:SOP50P310X90-8N")
     )
     (path "/cc781fc4-5754-4e87-a81e-a175b2207ad4"

Commit message: Add files via upload
Connections:
- net CANH renamed CAN+
- net CANL renamed CAN-
Changed lines of the file:
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@@
     (effects (font (size 1.5 1.5) (thickness 0.3) bold) (justify left bottom))
   )
+  (label "CAN+" (at 34.29 100.33 0)
+    (effects (font (size 1.27 1.27)) (justify left bottom))
+  )
+  (label "CAN+" (at 105.41 106.68 0)
+    (effects (font (size 1.27 1.27)) (justify left bottom))
+  )
+  (label "CAN-" (at 105.41 111.76 0)
+    (effects (font (size 1.27 1.27)) (justify left bottom))
+  )
+  (label "CAN-" (at 34.29 102.87 0)
+    (effects (font (size 1.27 1.27)) (justify left bottom))
+  )
   (global_label "M2" (shape input) (at 270.51 30.48 180) (fields_autoplaced)
     (effects (font (size 1.27 1.27)) (justify right))
@@
     (effects (font (size 1.27 1.27)) (justify right))
   )
+  (hierarchical_label "TX_CAN" (shape input) (at 66.04 104.14 180)
+    (effects (font (size 1.27 1.27)) (justify right))
+  )
   (hierarchical_label "PGC" (shape input) (at 189.23 49.53 0)
     (effects (font (size 1.27 1.27)) (justify left))
   )
+  (hierarchical_label "RX_CAN" (shape input) (at 66.04 106.68 180)
+    (effects (font (size 1.27 1.27)) (justify right))
+  )
   (hierarchical_label "SCL1" (shape input) (at 81.28 162.56 180)
     (effects (font (size 1.27 1.27)) (justify right))
@@
     (effects (font (size 1.27 1.27)) (justify right))
   )
-  (hierarchical_label "CANL" (shape input) (at 105.41 111.76 0)
-    (effects (font (size 1.27 1.27)) (justify left))
-  )
-  (hierarchical_label "CANH" (shape input) (at 105.41 106.68 0)
-    (effects (font (size 1.27 1.27)) (justify left))
-  )
   (hierarchical_label "SDA1" (shape input) (at 81.28 177.8 180)
     (effects (font (size 1.27 1.27)) (justify right))
@@
     (effects (font (size 1.27 1.27)) (justify left))
   )
-  (hierarchical_label "CANL" (shape input) (at 34.29 102.87 0)
-    (effects (font (size 1.27 1.27)) (justify left))
-  )
   (hierarchical_label "RESET" (shape input) (at 127 35.56 90)
     (effects (font (size 1.27 1.27)) (justify left))
@@
     (effects (font (size 1.27 1.27)) (justify left))
   )
-  (hierarchical_label "CANH" (shape input) (at 34.29 100.33 0)
-    (effects (font (size 1.27 1.27)) (justify left))
-  )
   (hierarchical_label "PMW_5V" (shape input) (at 128.27 82.55 180)
     (effects (font (size 1.27 1.27)) (justify right))
   )
-  (hierarchical_label "RX_CAN" (shape input) (at 66.04 106.68 180)
-    (effects (font (size 1.27 1.27)) (justify right))
-  )
   (hierarchical_label "PMW_5V" (shape input) (at 186.69 138.43 180)
     (effects (font (size 1.27 1.27)) (justify right))
   )
-  (hierarchical_label "TX_CAN" (shape input) (at 66.04 104.14 180)
-    (effects (font (size 1.27 1.27)) (justify right))
-  )

Commit message: Add files via upload
Connections:
- net GND: now also Q2.2 (E)
- net M1: now also R18.2, Rshunt1.1
- net VBAT: now also D6.1 (K), D7.1 (K), K2.2, K3.2
- removed net Relé_Out: Q2.2 (E), R18.2, Rshunt1.1

Commit message: Add files via upload
Parts:
- C13, C3, C8: footprint Capacitor_THT:C_Radial_D4.0mm_H5.0mm_P1.50mm -> Capacitor_SMD:C_1206_3216Metric
- U2: footprint Package_DIP:DIP-8_W7.62mm -> Llibreria_projecte:TRANSCEIVER_SMD
- U3, U4: footprint BQ_Library:TO254P1054X470X1955-3 -> BQ_Library:TO-220
- U5: footprint Llibreria_Projecte_Maleter:SON50P400X400X100-13N -> Llibreria_projecte:SON50P400X400X100-13N
Connections:
- net Heater: now also U6.3 (RA1/AN1); no longer U6.25 (RB4)
- net INTERRP: now also U6.23 (RB2/CANTX/INT2); no longer U6.2 (RA0/AN0/CVREF)
Changed lines of the file:
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@@
   )
   (no_connect (at 30.48 105.41))
-  (no_connect (at 128.27 59.69))
+  (no_connect (at 128.27 69.85))
   (no_connect (at 189.23 55.88))
   (no_connect (at 30.48 113.03))
@@
   (no_connect (at 128.27 44.45))
   (no_connect (at 30.48 95.25))
-  (no_connect (at 128.27 52.07))
+  (no_connect (at 128.27 57.15))
   (no_connect (at 189.23 44.45))
   (no_connect (at 66.04 111.76))
@@
     (stroke (width 0) (type default) (color 0 0 0 0))
   )
-  (wire (pts (xy 127 69.85) (xy 128.27 69.85))
-    (stroke (width 0) (type default) (color 0 0 0 0))
-  )
   (wire (pts (xy 213.36 137.16) (xy 210.82 137.16))
     (stroke (width 0) (type default) (color 0 0 0 0))
@@
     (stroke (width 0) (type default) (color 0 0 0 0))
   )
-  (wire (pts (xy 127 57.15) (xy 128.27 57.15))
-    (stroke (width 0) (type default) (color 0 0 0 0))
-  )
   (wire (pts (xy 132.08 147.32) (xy 132.08 148.59))
     (stroke (width 0) (type default) (color 0 0 0 0))
@@
     )
   )
-  (global_label "INTERRP" (shape input) (at 127 57.15 180) (fields_autoplaced)
+  (global_label "INTERRP" (shape input) (at 128.27 52.07 180) (fields_autoplaced)
     (effects (font (size 1.27 1.27)) (justify right))
-    (property "Intersheet References" "${INTERSHEET_REFS}" (id 0) (at 116.725 57.0706 0)
+    (property "Intersheet References" "${INTERSHEET_REFS}" (id 0) (at 117.995 51.9906 0)
       (effects (font (size 1.27 1.27)) (justify right) hide)
     )
@@
     (effects (font (size 1.27 1.27)) (justify left))
   )
-  (hierarchical_label "Heater" (shape input) (at 127 69.85 180)
+  (hierarchical_label "Heater" (shape input) (at 128.27 59.69 180)
     (effects (font (size 1.27 1.27)) (justify right))
   )
@@
     (property "Reference" "U5" (id 0) (at 99.06 134.62 0))
     (property "Value" "FDC2212QDNTTQ1" (id 1) (at 99.06 137.16 0))
-    (property "Footprint" "Llibreria_Projecte_Maleter:SON50P400X400X100-13N" (id 2) (at 99.06 162.56 0)
+    (property "Footprint" "Llibreria_projecte:SON50P400X400X100-13N" (id 2) (at 99.06 162.56 0)
       (effects (font (size 1.27 1.27)) (justify bottom) hide)
     )
@@
       (effects (font (size 1.27 1.27)) (justify left))
     )
-    (property "Footprint" "Capacitor_THT:C_Radial_D4.0mm_H5.0mm_P1.50mm" (id 2) (at 69.85 96.52 0)
+    (property "Footprint" "Capacitor_SMD:C_1206_3216Metric" (id 2) (at 69.85 96.52 0)
       (effects (font (size 1.27 1.27)) hide)
     )
@@
       (effects (font (size 1.27 1.27)) (justify left))
     )
-    (property "Footprint" "Capacitor_THT:C_Radial_D4.0mm_H5.0mm_P1.50mm" (id 2) (at 104.14 109.22 0)
+    (property "Footprint" "Capacitor_SMD:C_1206_3216Metric" (id 2) (at 104.14 109.22 0)
       (effects (font (size 1.27 1.27)) hide)
     )
@@
     (property "Reference" "U4" (id 0) (at 82.55 54.61 0))
     (property "Value" "LM1117-3.3" (id 1) (at 82.55 52.07 0))
-    (property "Footprint" "BQ_Library:TO254P1054X470X1955-3" (id 2) (at 82.55 54.61 0)
+    (property "Footprint" "BQ_Library:TO-220" (id 2) (at 82.55 54.61 0)
       (effects (font (size 1.27 1.27)) hide)
     )
@@
     (property "Reference" "U3" (id 0) (at 82.55 25.4 0))
     (property "Value" "LM1117-5.0" (id 1) (at 82.55 21.59 0))
-    (property "Footprint" "BQ_Library:TO254P1054X470X1955-3" (id 2) (at 82.55 25.4 0)
+    (property "Footprint" "BQ_Library:TO-220" (id 2) (at 82.55 25.4 0)
       (effects (font (size 1.27 1.27)) hide)
     )
@@
       (effects (font (size 1.27 1.27)) (justify left))
     )
-    (property "Footprint" "Package_DIP:DIP-8_W7.62mm" (id 2) (at 78.74 121.92 0)
+    (property "Footprint" "Llibreria_projecte:TRANSCEIVER_SMD" (id 2) (at 78.74 121.92 0)
       (effects (font (size 1.27 1.27) italic) hide)
     )
@@
       (effects (font (size 1.27 1.27)) (justify left))
     )
-    (property "Footprint" "Capacitor_THT:C_Radial_D4.0mm_H5.0mm_P1.50mm" (id 2) (at 198.12 36.83 0)
+    (property "Footprint" "Capacitor_SMD:C_1206_3216Metric" (id 2) (at 198.12 36.83 0)
       (effects (font (size 1.27 1.27)) hide)
     )
@@
     )
     (path "/4faaaf16-8692-49c6-9f28-55697217bb23"
-      (reference "C3") (unit 1) (value "100nF") (footprint "Capacitor_THT:C_Radial_D4.0mm_H5.0mm_P1.50mm")
+      (reference "C3") (unit 1) (value "100nF") (footprint "Capacitor_SMD:C_1206_3216Metric")
     )
     (path "/6b7e06ad-7a47-4abb-b269-546d2ae88f4e"
@@
     )
     (path "/75505ded-0440-45cd-a678-1c0fdb16a964"
-      (reference "C8") (unit 1) (value "100pF") (footprint "Capacitor_THT:C_Radial_D4.0mm_H5.0mm_P1.50mm")
+      (reference "C8") (unit 1) (value "100pF") (footprint "Capacitor_SMD:C_1206_3216Metric")
     )
     (path "/eded7ed9-1d3f-47c6-99e9-1bf5e7bf7cdd"
@@
     )
     (path "/d3df1af1-aa9f-404d-b57e-4d9f35f9b12d"
-      (reference "C13") (unit 1) (value "100nF") (footprint "Capacitor_THT:C_Radial_D4.0mm_H5.0mm_P1.50mm")
+      (reference "C13") (unit 1) (value "100nF") (footprint "Capacitor_SMD:C_1206_3216Metric")
     )
     (path "/77c4d080-93d1-4e51-baba-86a5b3b4f814"
@@
     )
     (path "/cc781fc4-5754-4e87-a81e-a175b2207ad4"
-      (reference "U2") (unit 1) (value "MCP2551-I-P") (footprint "Package_DIP:DIP-8_W7.62mm")
+      (reference "U2") (unit 1) (value "MCP2551-I-P") (footprint "Llibreria_projecte:TRANSCEIVER_SMD")
     )
     (path "/8ae3d050-26a8-49c5-9503-ad56288cb2da"
-      (reference "U3") (unit 1) (value "LM1117-5.0") (footprint "BQ_Library:TO254P1054X470X1955-3")
+      (reference "U3") (unit 1) (value "LM1117-5.0") (footprint "BQ_Library:TO-220")
     )
     (path "/841d09d8-6429-40bd-8232-daf985229c58"
-      (reference "U4") (unit 1) (value "LM1117-3.3") (footprint "BQ_Library:TO254P1054X470X1955-3")
+      (reference "U4") (unit 1) (value "LM1117-3.3") (footprint "BQ_Library:TO-220")
     )
     (path "/32a96933-8c99-4093-9a61-0f82e9225116"
-      (reference "U5") (unit 1) (value "FDC2212QDNTTQ1") (footprint "Llibreria_Projecte_Maleter:SON50P400X400X100-13N")
+      (reference "U5") (unit 1) (value "FDC2212QDNTTQ1") (footprint "Llibreria_projecte:SON50P400X400X100-13N")
     )
     (path "/992a5159-c17d-41cf-b261-ccbf235da20d"

Commit message: Add files via upload
Parts:
- added C15, C16: 0.1 uF, Capacitor_SMD:C_0805_2012Metric_Pad1.18x1.45mm_HandSolder, symbol Device:C_Small
- C6, C7: footprint Capacitor_THT:C_Radial_D4.0mm_H5.0mm_P1.50mm -> Capacitor_SMD:C_1206_3216Metric
- R22: value 80k -> 120k
- U6: footprint Llibreria_Projecte_Maleter:DIP787W45P254L3556H508Q28 -> Llibreria_projecte:MICROSMD
- Y1: footprint Crystal:Crystal_HC49-4H_Vertical -> Llibreria_projecte:CRISTALL
Connections:
- net +VCC1: now also R20.1, C16.1
- net +VCC2: now also C15.1; no longer R20.1
- net GND: now also C15.2, C16.2
- net INTERRP: now also U6.26 (RB5/PGM); no longer U6.23 (RB2/CANTX/INT2)
- net Relé1: now also U6.24 (RB3/CANRX); no longer U6.11 (RC0/T1OSO/T1CK1)
- net Relé2: now also U6.16 (RC5/SDO); no longer U6.12 (RC1/T1OSI)
