File: Layout_Maleter.kicad_pcb (KiCad board)
At the start: 2 copper layers, 64 parts, among them J1 Conn_01x02, J2 DB9_Male, J3 Conn_01x02, J4 Conn_01x02, J5 Conn_01x06_Fem, J6 Conn_Male, J7 Conn_01x02, K1 ADW11, K2 1393280-5, K3 1393280-5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

Commit message: Add files via upload
Parts:
- added C14: 100 nF, Capacitor_SMD:C_0805_2012Metric, F.Cu at (413.0, 129.1)
- added D8: 1N4002, Diode_THT:D_5W_P10.16mm_Horizontal, F.Cu at (149.8, 151.8)
- added R14: 60k, Resistor_SMD:R_1206_3216Metric, F.Cu at (141.0, 86.4)
- added R16: 10k, Resistor_SMD:R_1206_3216Metric, F.Cu at (140.7, 88.9)
- added R23: 60k, Resistor_SMD:R_1206_3216Metric, F.Cu at (140.7, 93.5)
- added R24: 10k, Resistor_SMD:R_1206_3216Metric, F.Cu at (140.8, 96.5)
- added R4: 60k, Resistor_SMD:R_1206_3216Metric, F.Cu at (123.5, 101.6)
- added R5: 10k, Resistor_SMD:R_1206_3216Metric, F.Cu at (129.5, 103.1)
- moved Q2 4.62 mm to (146.1, 87.0)
- moved Q3 4.62 mm to (146.1, 94.0)
Connections:
- net VOUT renamed INTERRP
- C1 pad 2: +VCC2 -> Net-(C1-Pad2)
- C10 pad 2: +VCC2 -> GND
- C13 pad 2: +VCC2 -> GND
- C2 pad 2: +VCC2 -> Net-(C2-Pad2)
- C3 pad 2: +VCC2 -> GND
- C4 pad 2: +VCC2 -> GND
- C5 pad 2: +VCC2 -> GND
- C6 pad 2: +VCC2 -> GND
- C7 pad 2: +VCC2 -> GND
- C9 pad 2: +VCC2 -> GND
- D3 pad 1: +VCC2 -> GND
- D4 pad 1: +VCC2 -> GND
- D5 pad 1: +VCC2 -> GND
- D6 pad 1: VBAT -> Net-(D6-Pad1)
- D7 pad 1: VBAT -> Net-(K3-Pad2)
- J2 pad 4: +VCC2 -> GND
- J3 pad 1: +VCC2 -> GND
- J4 pad 1: +VCC2 -> GND
- J5 pad 1: //MCLR -> /RESET
- K2 pad 2: VBAT -> Net-(D6-Pad1)
- K2 pad 3: M1 -> VBAT
- K2 pad 4: VBAT -> M1
- K3 pad 2: VBAT -> Net-(K3-Pad2)
- K3 pad 3: M2 -> VBAT
- K3 pad 4: VBAT -> M2
- L1 pad 2: +VCC2 -> Net-(C1-Pad2)
- L2 pad 2: +VCC2 -> Net-(C2-Pad2)
- Q1 pad 1: /PMW_5V -> Net-(Q1-Pad1)
- Q2 pad 1: /Relé1 -> Net-(Q2-Pad1)
- Q3 pad 1: /Relé2 -> Net-(Q3-Pad1)
- Q3 pad 2: +VCC2 -> GND
- R1 pad 2: +VCC2 -> /SCL1
- R3 pad 2: +VCC2 -> /SDA1
- R6 pad 2: /SCL2 -> Net-(R6-Pad2)
- R7 pad 1: +VCC2 -> GND
- R8 pad 2: /SCL2 -> /SDA2
- S2 pad 4: +VCC2 -> GND
- U1 pad 1: +VCC2 -> GND
- U1 pad 3: +VCC2 -> /SCL1
- U1 pad 4: +VCC2 -> /SDA1
- U1 pad 5: /SCL2 -> /SDA2
- U1 pad 7: /SCL2 -> Net-(R6-Pad2)
- U1 pad 8: /SCL2 -> Net-(R6-Pad2)
- U2 pad 2: +VCC2 -> GND
- U2 pad 5: Net-(R4-Pad1) -> unconnected-(U2-Pad5)
- U5 pad 1: +VCC2 -> /SCL1
- U5 pad 10: +VCC2 -> Net-(C1-Pad2)
- U5 pad 12: +VCC2 -> Net-(C2-Pad2)
- U5 pad 2: +VCC2 -> /SDA1
- U5 pad 3: unconnected-(U5-Pad3) -> GND
- U5 pad 8: +VCC2 -> GND
- U6 pad 1: //MCLR -> /RESET
- U6 pad 15: /SCL2 -> /SDA2
- U6 pad 19: +VCC2 -> GND
- U6 pad 8: +VCC2 -> GND
- U7 pad 8: +VCC1 -> Net-(U7-Pad8)
Routing:
- net Net-(K1-Pad1): track 10.5 -> 40.0 mm
- net Net-(Q1-Pad1): track 0.00 -> 25.2 mm
- net /RESET: track 28.5 -> 51.9 mm
- net /PMW_5V: track 30.8 -> 7.71 mm
- net M2: track 30.8 -> 45.5 mm
- net /Relé_Out: track 16.3 -> 6.15 mm, vias 1 -> 0
- net //MCLR: track 8.28 -> 0.00 mm
- net M1: track 16.9 -> 24.9 mm
- net Net-(Q3-Pad1): track 0.00 -> 6.46 mm
- net Net-(D6-Pad1): track 0.00 -> 5.90 mm
- net Net-(Q2-Pad1): track 0.00 -> 5.46 mm
- net Net-(K3-Pad2): track 0.00 -> 5.34 mm
- net Net-(D6-Pad2): track 24.0 -> 20.1 mm
- net /Relé2: track 14.9 -> 11.2 mm
- net VBAT: track 87.5 -> 86.1 mm, vias 1 -> 0
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
Commit message: Add files via upload
Parts:
- added U3: LM1117-5.0, BQ_Library:TO254P1054X470X1955-3, F.Cu at (170.2, 58.4)
- added U4: LM1117-3.3, BQ_Library:TO254P1054X470X1955-3, F.Cu at (170.2, 73.7)
- moved D5 291.7 mm to (116.8, 76.2)
- moved R15 283.1 mm to (124.5, 76.2), turned to 90 degrees
- moved U1 259.9 mm to (157.5, 88.6), turned to 180 degrees
- moved C5 259.8 mm to (162.6, 73.7), turned to -90 degrees
- moved C4 248.0 mm to (162.6, 58.4), turned to 90 degrees
- moved C6 243.4 mm to (177.8, 61.0)
- moved R10 232.4 mm to (182.9, 61.0), turned to -90 degrees
- moved C2 222.4 mm to (175.3, 88.9), turned to 180 degrees
- moved U5 221.2 mm to (165.1, 91.4)
- moved C7 216.3 mm to (177.8, 73.7)
- moved C1 215.4 mm to (175.3, 96.5), turned to 180 degrees
- moved J4 213.5 mm to (182.9, 86.4)
- moved D4 209.1 mm to (180.3, 81.3), turned to 90 degrees
- moved J3 207.1 mm to (182.9, 96.5), turned to 180 degrees
- moved D1 204.3 mm to (162.6, 66.0)
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Routing:
- net Net-(C1-Pad1): track 0.00 -> 19.8 mm
- net Net-(C2-Pad1): track 0.00 -> 18.7 mm
- net Net-(C5-Pad1): track 0.00 -> 15.2 mm
- net Net-(D6-Pad2): track 20.1 -> 35.3 mm
- net M1: track 24.9 -> 38.2 mm
- net Net-(C4-Pad1): track 0.00 -> 12.1 mm
- net Net-(C2-Pad2): track 0.00 -> 11.0 mm
- net Net-(C1-Pad2): track 0.00 -> 9.40 mm
- net /SCL1: track 0.00 -> 6.15 mm
- net Net-(D5-Pad2): track 0.00 -> 5.69 mm
- net Net-(D3-Pad2): track 0.00 -> 4.67 mm
- net Net-(D4-Pad2): track 0.00 -> 4.67 mm
- net Net-(R15-Pad1): track 0.00 -> 4.66 mm
- net VBAT: track 86.1 -> 82.6 mm
- net M2: track 45.5 -> 47.4 mm
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
Commit message: Add files via upload
Parts:
- C14: moved to B.Cu
- U1: footprint Llibreria_Projecte_Maleter:TCA39306DTMR -> Llibreria_Projecte_Maleter:SOP50P310X90-8N
- moved C14 313.3 mm to (106.5, 64.0), turned to 180 degrees
- moved C3 311.0 mm to (115.0, 90.0), turned to 180 degrees
- moved R7 302.2 mm to (105.0, 105.0), turned to 90 degrees
- moved C8 299.0 mm to (101.6, 97.3), turned to 90 degrees
- moved R12 284.8 mm to (106.6, 97.3), turned to -90 degrees
- moved U2 276.3 mm to (118.6, 101.8), turned to 180 degrees
- moved C13 270.9 mm to (141.2, 78.0)
- moved R9 267.0 mm to (154.0, 73.5)
- moved J2 262.4 mm to (85.0, 95.0), turned to -90 degrees
- moved R3 259.8 mm to (167.0, 85.0), turned to 180 degrees
- moved R4 259.5 mm to (125.0, 110.0), turned to 90 degrees
- moved C10 257.3 mm to (160.0, 96.0), turned to -90 degrees
- moved C9 249.1 mm to (163.0, 95.8), turned to -90 degrees
- moved R5 246.5 mm to (125.0, 115.0), turned to -90 degrees
- moved R6 242.3 mm to (154.0, 77.8)
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Connections:
- R4 pad 2: +VCC1 -> Net-(Q1-Pad1)
- R5 pad 1: +VCC2 -> Net-(R4-Pad1)
- R5 pad 2: Net-(R4-Pad1) -> GND
Routing:
- net /Relé_Out: track 6.15 -> 67.4 mm
- net /SCL2: track 0.00 -> 55.9 mm, vias 0 -> 3
- net /SDA2: track 0.00 -> 39.4 mm, vias 0 -> 5
- net VBAT: track 82.6 -> 117.7 mm, vias 0 -> 2
- net /INTB: track 0.00 -> 32.5 mm, vias 0 -> 1
- net /SD: track 0.00 -> 31.7 mm, vias 0 -> 1
- net /CANL: track 0.00 -> 31.3 mm
- net /CANH: track 0.00 -> 27.0 mm
- net GND: track 0.00 -> 25.8 mm, vias 0 -> 4
- net /TX_CAN: track 0.00 -> 22.8 mm
- net +VCC2: track 0.00 -> 22.2 mm, vias 0 -> 3
- net /RX_CAN: track 0.00 -> 19.9 mm
- net +VCC1: track 0.00 -> 18.3 mm
- net Net-(R6-Pad2): track 0.00 -> 12.0 mm, vias 0 -> 2
- net Net-(C14-Pad2): track 0.00 -> 10.2 mm
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- added copper zone on In1.Cu, net +VCC1
- added copper zone on In2.Cu, net +VCC2
- added copper zone on F.Cu, net GND
Other:
- board outline added: 114.5 x 120.5 mm
- copper layers 2 -> 4
