File: Layout_Maleter.kicad_pcb (KiCad board)
At the start: 4 copper layers, 79 x 67.2 mm, 80 parts, among them J1 Conn_01x02, J2 DB9_Male, J3 Conn_01x02, J4 Conn_01x02, J5 Conn_01x06_Fem, J6 Conn_Male, J7 Conn_01x02, K1 ADW11, K2 1393280-5, K3 1393280-5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

Commit message: Add files via upload
Other:
- board text added: "+"
- board text added: "-"
- board text added: "HEATER"
- board text added: "MOTOR"
- board text added: "Prog. Conn"
Changed lines of the file:
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@@
     (pad "28" smd rect locked (at 4.675 -8.255 90) (size 0.65 1.85) (layers "F.Cu" "F.Paste" "F.Mask")
       (net 26 "/PGD") (pinfunction "RB7/PGD") (pintype "bidirectional"))
-    (model "PIC18F2580-E_SO.stp"
+    (model "C:/Users/Jan (SUS)/Desktop/Disseny Kicad/PIC18F258-I_SO.stp"
+      (offset (xyz 0 0 0))
+      (scale (xyz 1 1 1))
+      (rotate (xyz 0 0 0))
+    )
+    (model "C:/Users/Jan (SUS)/Desktop/Disseny Kicad/PIC18F2580-E_SO.mod"
       (offset (xyz 0 0 0))
       (scale (xyz 1 1 1))
@@
     (tags "mounting hole 3.2mm m3 din965")
     (attr exclude_from_pos_files exclude_from_bom)
-    (fp_text reference "REF**" (at 0 -2.75) (layer "F.SilkS")
+    (fp_text reference "REF**" (at 0 -2.75) (layer "Dwgs.User")
       (effects (font (size 1 1) (thickness 0.15)))
     )
@@
     (tags "mounting hole 3.2mm m3 din965")
     (attr exclude_from_pos_files exclude_from_bom)
-    (fp_text reference "REF**" (at 0 -3.8) (layer "F.SilkS")
+    (fp_text reference "REF**" (at 0 -3.8) (layer "Dwgs.User")
       (effects (font (size 1 1) (thickness 0.15)))
     )
@@
     (fp_arc (start 0.196073 5.57) (mid -0.832387 5.195671) (end -1.379619 4.247837) (layer "F.Fab") (width 0.1))
     (fp_arc (start 11.783194 -2.73) (mid 13.00887 -2.158462) (end 13.358886 -0.852163) (layer "F.Fab") (width 0.1))
-    (fp_arc (start 12.459619 4.247837) (mid 11.912387 5.19567) (end 10.883927 5.57) (layer "F.Fab") (width 0.1))
+    (fp_arc (start 12.459619 4.247837) (mid 11.912387 5.195673) (end 10.883927 5.57) (layer "F.Fab") (width 0.1))
     (pad "1" thru_hole rect (at 0 0 90) (size 1.6 1.6) (drill 1) (layers *.Cu *.Mask)
       (net 17 "unconnected-(J2-Pad1)") (pinfunction "1") (pintype "passive+no_connect"))
@@
     (tags "mounting hole 3.2mm m3 din965")
     (attr exclude_from_pos_files exclude_from_bom)
-    (fp_text reference "REF**" (at 0 -3.8) (layer "F.SilkS")
+    (fp_text reference "REF**" (at 0 -3.8) (layer "User.1")
       (effects (font (size 1 1) (thickness 0.15)))
     )
@@
     (tags "mounting hole 3.2mm m3 din965")
     (attr exclude_from_pos_files exclude_from_bom)
-    (fp_text reference "REF**" (at 0.15 -2.45) (layer "F.SilkS")
+    (fp_text reference "REF**" (at 0.15 -2.45) (layer "Dwgs.User")
       (effects (font (size 1 1) (thickness 0.15)))
     )
@@
   )
   (gr_rect (start 100.7 47.6) (end 179.7 114.8) (layer "Edge.Cuts") (width 0.05) (fill none))
-  (gr_text "DESIGNED BY \nBethany Quintero/Jan Castillo\nUniversitat de Barcelona\nV3" (at 134.7 51.5) (layer "F.SilkS")
+  (gr_text "DESIGNED BY \nBethany Quintero/Jan Castillo\nUniversitat de Barcelona\nV3" (at 134.6 50.8) (layer "F.SilkS")
     (effects (font (size 1 0.7) (thickness 0.17)))
   )
+  (gr_text "Prog. Conn\n" (at 133 54.6) (layer "F.SilkS")
+    (effects (font (size 1 1) (thickness 0.15)))
+  )
+  (gr_text "+\n" (at 144.8 111.2) (layer "F.SilkS")
+    (effects (font (size 1 1) (thickness 0.15)))
+  )
+  (gr_text "+" (at 178.2 100) (layer "F.SilkS")
+    (effects (font (size 1.5 1.5) (thickness 0.3)))
+  )
+  (gr_text "HEATER\n" (at 146.4 113.2) (layer "F.SilkS")
+    (effects (font (size 1 1) (thickness 0.15)))
+  )
+  (gr_text "-" (at 147.6 111.2) (layer "F.SilkS")
+    (effects (font (size 1 1) (thickness 0.15)))
+  )
+  (gr_text "MOTOR\n" (at 175 105.6) (layer "F.SilkS")
+    (effects (font (size 1.5 1.5) (thickness 0.3)))
+  )
+  (gr_text "-" (at 178.2 102.8) (layer "F.SilkS")
+    (effects (font (size 1.5 1.5) (thickness 0.3)))
+  )
   (segment (start 168.90048 62.14952) (end 168.90048 55.80048) (width 0.25) (layer "F.Cu") (net 1))

Commit message: Add files via upload
Routing:
- added copper zone on B.Cu, net GND

Commit message: Add files via upload
Parts:
- removed C7: 10uF, Capacitor_SMD:C_1206_3216Metric
- moved FB2 72.4 mm to (175.1, 69.4), turned to -90 degrees
- moved FB1 50.4 mm to (109.1, 110.8)
- moved D1 11.4 mm to (128.1, 110.8), turned to 0 degrees
- moved R18 10.5 mm to (154.4, 65.0), turned to -90 degrees
- moved L1 6.10 mm to (168.8, 68.5), turned to 90 degrees
- moved C4 5.19 mm to (127.6, 106.6)
- moved D4 4.74 mm to (171.3, 80.1), turned to 180 degrees
- moved U2 4.00 mm to (122.9, 81.9), turned to -90 degrees
- moved J3 3.90 mm to (176.2, 65.6)
- moved K3 3.65 mm to (164.0, 104.8)
- moved R11 3.38 mm to (168.9, 74.4), turned to -90 degrees
- moved R16 3.30 mm to (142.4, 72.0)
- moved C5 3.28 mm to (176.2, 82.3)
- moved D2 3.03 mm to (175.7, 85.2)
- moved J1 2.97 mm to (165.6, 112.7)
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Routing:
- net M1: track 71.7 -> 53.7 mm
- net Net-(R18-Pad1): track 7.78 -> 22.0 mm
- net Net-(C4-Pad1): track 18.3 -> 8.25 mm
- net GND: track 54.2 -> 44.2 mm, vias 47 -> 73
- net /RX_CAN: track 12.8 -> 22.2 mm
- net Net-(C1-Pad1): track 19.0 -> 26.9 mm
- net Net-(C1-Pad2): track 20.7 -> 14.1 mm
- net /CAN-: track 24.9 -> 20.7 mm
- net /CAN+: track 26.2 -> 22.4 mm
- net +VCC1: track 32.6 -> 29.5 mm, vias 7 -> 11
- net Net-(C2-Pad2): track 9.72 -> 6.81 mm
- net Net-(Q2-Pad1): track 8.81 -> 11.2 mm
- net Net-(D7-Pad2): track 35.1 -> 36.5 mm
- net /TX_CAN: track 14.7 -> 16.0 mm
- net Net-(D6-Pad2): track 27.4 -> 28.5 mm
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- added copper zone on In1.Cu, net GND
- added copper zone on In2.Cu, net GNDPWR
Other:
- board text added: "DESIGNED BY Bethany Quintero/Jan Castillo Universitat de Barcelona V4"
- board text removed: "DESIGNED BY Bethany Quintero/Jan Castillo Universitat de Barcelona V3"
